Commit message: feat: dual arm trajectory execution working, now smilei_dual_arm_ik package has its configuration files uploaded, updated joint limits in remote_teleoperation state

File: src/smilei_dual_arm_ik/urdf/single_arm_parametric.urdf.xacro (robot description, xacro)
@@ -26,5 +26,5 @@
   <xacro:arg name="link2_width" default="0.20"/>
   <xacro:property name="link2_width" value="$(arg link2_width)"/>
-  <xacro:arg name="link3_length" default="-0.2"/>
+  <xacro:arg name="link3_length" default="0.2"/>
   <xacro:property name="link3_length" value="$(arg link3_length)"/>
   <xacro:arg name="link4_length" default="-0.08"/>
@@ -142,5 +142,5 @@
     <parent link="link_2"/>
     <child link="link_3"/>
-    <origin xyz="0 ${link2_length} ${link2_width}" rpy="${PI_2} 0 0"/>
+    <origin xyz="0 ${link2_length} ${link2_width}" rpy="${-PI_2} ${-PI_2} 0"/>
     <axis xyz="0 0 1"/>
     <limit lower="${joint2_lower}" upper="${joint2_upper}" effort="${joint2_effort}" velocity="${joint2_velocity}"/>
@@ -166,5 +166,5 @@
     <parent link="link_3"/>
     <child link="link_4"/>
-    <origin xyz="0 0 ${link3_length}" rpy="${PI_2} 0 0"/>
+    <origin xyz="0 0 ${link3_length}" rpy="${PI_2} 0 ${PI_2}"/>
     <axis xyz="0 0 1"/>
     <limit lower="${joint3_lower}" upper="${joint3_upper}" effort="${joint3_effort}" velocity="${joint3_velocity}"/>
@@ -190,5 +190,5 @@
     <parent link="link_4"/>
     <child link="end_effector"/>
-    <origin xyz="0 ${link4_length + ee_offset} 0" rpy="-${PI_2} 0 -${PI_2}"/>
+    <origin xyz="0 ${link4_length + ee_offset} 0" rpy="${PI_2} 0 ${PI_2}"/>
   </joint>
   <link name="end_effector">
